Commit message: Changed angle for the finger joints to 50 degrees

File: barrett_hand_description/urdf/bh280.urdf.xacro (robot description, xacro)
@@ -391,5 +391,5 @@
 			<parent link="${name}_finger_13_link"/>
 			<child link="${name}_finger_14_link"/>
-			<origin xyz="0 0 0" rpy="0 0 0.698132" />
+			<origin xyz="0 0 0" rpy="0 0 0.872665" />
 		</joint>
 		<link name="${name}_finger_14_link"/>
@@ -397,5 +397,5 @@
 			<parent link="${name}_finger_23_link"/>
 			<child link="${name}_finger_24_link"/>
-			<origin xyz="0 0 0" rpy="0 0 0.698132" />
+			<origin xyz="0 0 0" rpy="0 0 0.872665" />
 		</joint>
 		<link name="${name}_finger_24_link"/>
@@ -403,5 +403,5 @@
 			<parent link="${name}_finger_33_link"/>
 			<child link="${name}_finger_34_link"/>
-			<origin xyz="0 0 0" rpy="0 0 0.698132" />
+			<origin xyz="0 0 0" rpy="0 0 0.872665" />
 		</joint>
 		<link name="${name}_finger_34_link"/>
